Commit message: Relabel object set (17 objects) and exclude else_* from training (9-object set)
Second and third passes over the training object roster, following up on
GPU training results showing a clear reward gap for the geometrically
distinct new objects:

- Removed the procedurally-generated stair-shaped block_3 and all 4 ball_*
  objects (sphere, dodecahedron, icosahedron, ellipsoid) entirely -- they
  scored noticeably lower reward than the rest of the set.
- Promoted else_1 -> block_3 and else_5 -> block_5 (plain blocks, not the
  removed stair shape), renumbered the remaining else_2,3,4,6,7,8,9,10 down
  to else_1..else_8.
- Excluded else_1..else_8 from object_sets["C"] entirely, narrowing the
  active training roster to 9 curated objects (block_1..5, cylinder_1..4).
  Generalization beyond these is explicitly not a goal for this run; the
  else_* assets remain on disk/in asset_files_dict for possible future reuse.
- Regenerated tools/object_viewer.html's embedded mesh data and updated
  README.md to describe the three-pass object-set history.

Also recovers from an in-session bug in the first relabeling script (a
chained rename clobbered else_1..8 before this commit); the final state was
rebuilt via a safe copy-to-temp-name -> delete -> rename-to-final approach
and re-verified (mesh/urdf reference integrity, object_sets["C"] consistency,
py_compile).

File: assets/urdf/objects/block_3.urdf (robot description, URDF)
Before this commit: robot object, 1 links, 0 joints
Links:
- link object: geometry collision mesh filename=meshes/set2/block_3_0decompose.obj scale=.03 .03 .03; visual mesh filename=meshes/set2/block_3.obj scale=.03 .03 .03

File: assets/urdf/objects/block_5.urdf (robot description, URDF)
Before this commit: robot object, 1 links, 0 joints
Links:
- link object: geometry collision mesh filename=meshes/set2/block_5_0decompose.obj scale=.03 .03 .03; visual mesh filename=meshes/set2/block_5.obj scale=.03 .03 .03

File: assets/urdf/objects/else_1.urdf (robot description, URDF)
Before this commit: robot object, 1 links, 0 joints
Links:
- link object: geometry collision mesh filename=meshes/set2/else_1_0decompose.obj scale=.03 .03 .03; collision mesh filename=meshes/set2/else_1_1decompose.obj scale=.03 .03 .03

File: assets/urdf/objects/else_2.urdf (robot description, URDF)
Before this commit: robot object, 1 links, 0 joints
Links:
- link object: geometry collision mesh filename=meshes/set2/else_2_0decompose.obj scale=.03 .03 .03; collision mesh filename=meshes/set2/else_2_10decompose.obj scale=.03 .03 .03

File: assets/urdf/objects/else_3.urdf (robot description, URDF)
Before this commit: robot object, 1 links, 0 joints
Links:
- link object: geometry collision mesh filename=meshes/set2/else_3_0decompose.obj scale=.03 .03 .03; collision mesh filename=meshes/set2/else_3_1decompose.obj scale=.03 .03 .03

File: assets/urdf/objects/else_4.urdf (robot description, URDF)
Before this commit: robot object, 1 links, 0 joints
Links:
- link object: geometry collision mesh filename=meshes/set2/else_4_0decompose.obj scale=.03 .03 .03; visual mesh filename=meshes/set2/else_4.obj scale=.03 .03 .03

File: assets/urdf/objects/else_8.urdf (robot description, URDF)
Before this commit: robot object, 1 links, 0 joints
Links:
- link object: geometry collision mesh filename=meshes/set2/else_8_0decompose.obj scale=.03 .03 .03; collision mesh filename=meshes/set2/else_8_1decompose.obj scale=.03 .03 .03
