Commit message: Restore 9-object set, fix object init pose randomization, disable DR ramp
- Object set back to the 9 training objects "C" (block_1..5, cylinder_1..4).
  Eight are original in-hand-rotation objects renamed (matched by mesh
  geometry); cylinder_3 (decagon prism) restored from 3e0c2fe. The other 8
  original objects are removed. objSet default is now "C".
- Fix object initial pose randomization never reaching the sim: reset_idx
  re-set object mass via set_actor_rigid_body_properties, which on the GPU
  pipeline discards the root-state write made in the same step. Mass is now
  randomized once per env at creation.
- Initial pose randomization now always at full range (not DR-ramped):
  x/y ~ U(-1.5cm, 1.5cm), z ~ U(0, 1cm), yaw ~ U(-pi, pi)
  (objInitPosNoiseXY / objInitPosZLow / objInitPosZHigh).
- Progressive DR ramp disabled by default (drRampEnable: False), matching
  the 2026-10-20 rws2-randinit-zup run.
- evaluate_policy_per_object.py: drop zero-length episodes and record how
  many were dropped per object.
- players.py: read object count from env instead of a fixed objSet table.
- Regenerate object_viewer.html and update tools for the 9-object set.

Co-Authored-By: Claude Opus 5.5 <noreply@anthropic.com>

File: assets/urdf/objects/block_1.urdf (robot description, URDF)
Before this commit: robot object, 1 links, 0 joints
Links:
- link object: geometry collision mesh filename=meshes/set2/block_1_0decompose.obj scale=.03 .03 .03; visual mesh filename=meshes/set2/block_1.obj scale=.03 .03 .03

File: assets/urdf/objects/block_2.urdf (robot description, URDF)
Before this commit: robot object, 1 links, 0 joints
Links:
- link object: geometry collision mesh filename=meshes/set2/block_2_0decompose.obj scale=.03 .03 .03; collision mesh filename=meshes/set2/block_2_1decompose.obj scale=.03 .03 .03

File: assets/urdf/objects/block_3.urdf (robot description, URDF)
Before this commit: robot object, 1 links, 0 joints
Links:
- link object: geometry collision mesh filename=meshes/set2/block_3_0decompose.obj scale=.03 .03 .03; visual mesh filename=meshes/set2/block_3.obj scale=.03 .03 .03

File: assets/urdf/objects/block_4.urdf (robot description, URDF)
Before this commit: robot object, 1 links, 0 joints
Links:
- link object: geometry collision mesh filename=meshes/set2/block_4_0decompose.obj scale=.03 .03 .03; visual mesh filename=meshes/set2/block_4.obj scale=.03 .03 .03

File: assets/urdf/objects/block_5.urdf (robot description, URDF)
Before this commit: robot object, 1 links, 0 joints
Links:
- link object: geometry collision mesh filename=meshes/set2/block_5_0decompose.obj scale=.03 .03 .03; visual mesh filename=meshes/set2/block_5.obj scale=.03 .03 .03

File: assets/urdf/objects/cylinder_1.urdf (robot description, URDF)
Before this commit: robot object, 1 links, 0 joints
Links:
- link object: geometry collision mesh filename=meshes/set2/cylinder_1_0decompose.obj scale=.03 .03 .03; visual mesh filename=meshes/set2/cylinder_1.obj scale=.03 .03 .03

File: assets/urdf/objects/cylinder_2.urdf (robot description, URDF)
Before this commit: robot object, 1 links, 0 joints
Links:
- link object: geometry collision mesh filename=meshes/set2/cylinder_2_0decompose.obj scale=.03 .03 .03; collision mesh filename=meshes/set2/cylinder_2_1decompose.obj scale=.03 .03 .03

File: assets/urdf/objects/cylinder_4.urdf (robot description, URDF)
Before this commit: robot object, 1 links, 0 joints
Links:
- link object: geometry collision mesh filename=meshes/set2/cylinder_4_0decompose.obj scale=.03 .03 .03; visual mesh filename=meshes/set2/cylinder_4.obj scale=.03 .03 .03
